File: PCB/PCB.kicad_sch (KiCad schematic)
At the start: 78 parts, among them SW10 SW_Push, SW11 SW_Push, SW12 SW_Push, SW13 SW_Push, SW14 SW_Push, SW15 SW_Push, SW16 SW_Push, SW17 SW_Push, SW18 SW_Push, SW19 SW_Push, SW2 SW_Push, SW20 SW_Push, SW21 SW_Push, SW22 SW_Push, SW23 SW_Push, SW24 SW_Push, SW25 SW_Push, SW26 SW_Push, SW3 SW_Push, SW4 SW_Push, SW5 SW_Push, SW6 SW_Push, SW7 SW_Push, SW8 SW_Push, SW9 SW_Push, U1 COM-09032, U2 COM-09032

Commit message: fix the joystick footprint
Parts:
- U1, U2: footprint stno:XDCR_COM-09032 -> stno:PS4_joystick
Changed lines of the file:
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@@
 			)
 		)
-		(property "Footprint" "stno:XDCR_COM-09032"
+		(property "Footprint" "stno:PS4_joystick"
 			(at 143.51 35.56 0)
 			(effects
@@
 			)
 		)
-		(property "Footprint" "stno:XDCR_COM-09032"
+		(property "Footprint" "stno:PS4_joystick"
 			(at 191.77 35.56 0)
 			(effects

Commit message: hotswap switches fixed
Parts:
- SW10, SW11, SW12, SW13, SW14, SW15, SW16, SW17, SW18, SW19, SW2, SW20, SW21, SW22, SW23, SW24, SW25, SW26, SW3, SW4, SW5, SW6, SW7, SW8, SW9: footprint keebio:Kailh_MX_Socket-compat -> Library:hotswap
Changed lines of the file:
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@@
 			)
 		)
-		(property "Footprint" "keebio:Kailh_MX_Socket-compat"
+		(property "Footprint" "Library:hotswap"
 			(at 195.58 147.32 0)
 			(effects
@@
 			)
 		)
-		(property "Footprint" "keebio:Kailh_MX_Socket-compat"
+		(property "Footprint" "Library:hotswap"
 			(at 195.58 129.54 0)
 			(effects
@@
 			)
 		)
-		(property "Footprint" "keebio:Kailh_MX_Socket-compat"
+		(property "Footprint" "Library:hotswap"
 			(at 195.58 76.2 0)
 			(effects
@@
 			)
 		)
-		(property "Footprint" "keebio:Kailh_MX_Socket-compat"
+		(property "Footprint" "Library:hotswap"
 			(at 195.58 111.76 0)
 			(effects
@@
 			)
 		)
-		(property "Footprint" "keebio:Kailh_MX_Socket-compat"
+		(property "Footprint" "Library:hotswap"
 			(at 181.61 76.2 0)
 			(effects
@@
 			)
 		)
-		(property "Footprint" "keebio:Kailh_MX_Socket-compat"
+		(property "Footprint" "Library:hotswap"
 			(at 181.61 93.98 0)
 			(effects
@@
 			)
 		)
-		(property "Footprint" "keebio:Kailh_MX_Socket-compat"
+		(property "Footprint" "Library:hotswap"
 			(at 209.55 129.54 0)
 			(effects
@@
 			)
 		)
-		(property "Footprint" "keebio:Kailh_MX_Socket-compat"
+		(property "Footprint" "Library:hotswap"
 			(at 223.52 111.76 0)
 			(effects
@@
 			)
 		)
-		(property "Footprint" "keebio:Kailh_MX_Socket-compat"
+		(property "Footprint" "Library:hotswap"
 			(at 209.55 93.98 0)
 			(effects
@@
 			)
 		)
-		(property "Footprint" "keebio:Kailh_MX_Socket-compat"
+		(property "Footprint" "Library:hotswap"
 			(at 237.49 111.76 0)
 			(effects
@@
 			)
 		)
-		(property "Footprint" "keebio:Kailh_MX_Socket-compat"
+		(property "Footprint" "Library:hotswap"
 			(at 181.61 129.54 0)
 			(effects
@@
 			)
 		)
-		(property "Footprint" "keebio:Kailh_MX_Socket-compat"
+		(property "Footprint" "Library:hotswap"
 			(at 223.52 76.2 0)
 			(effects
@@
 			)
 		)
-		(property "Footprint" "keebio:Kailh_MX_Socket-compat"
+		(property "Footprint" "Library:hotswap"
 			(at 237.49 147.32 0)
 			(effects
@@
 			)
 		)
-		(property "Footprint" "keebio:Kailh_MX_Socket-compat"
+		(property "Footprint" "Library:hotswap"
 			(at 181.61 147.32 0)
 			(effects
@@
 			)
 		)
-		(property "Footprint" "keebio:Kailh_MX_Socket-compat"
+		(property "Footprint" "Library:hotswap"
 			(at 237.49 93.98 0)
 			(effects
@@
 			)
 		)
-		(property "Footprint" "keebio:Kailh_MX_Socket-compat"
+		(property "Footprint" "Library:hotswap"
 			(at 181.61 111.76 0)
 			(effects
@@
 			)
 		)
-		(property "Footprint" "keebio:Kailh_MX_Socket-compat"
+		(property "Footprint" "Library:hotswap"
 			(at 209.55 111.76 0)
 			(effects
@@
 			)
 		)
-		(property "Footprint" "keebio:Kailh_MX_Socket-compat"
+		(property "Footprint" "Library:hotswap"
 			(at 223.52 147.32 0)
 			(effects
@@
 			)
 		)
-		(property "Footprint" "keebio:Kailh_MX_Socket-compat"
+		(property "Footprint" "Library:hotswap"
 			(at 237.49 76.2 0)
 			(effects
@@
 			)
 		)
-		(property "Footprint" "keebio:Kailh_MX_Socket-compat"
+		(property "Footprint" "Library:hotswap"
 			(at 223.52 129.54 0)
 			(effects
@@
 			)
 		)
-		(property "Footprint" "keebio:Kailh_MX_Socket-compat"
+		(property "Footprint" "Library:hotswap"
 			(at 223.52 93.98 0)
 			(effects
@@
 			)
 		)
-		(property "Footprint" "keebio:Kailh_MX_Socket-compat"
+		(property "Footprint" "Library:hotswap"
 			(at 237.49 129.54 0)
 			(effects
@@
 			)
 		)
-		(property "Footprint" "keebio:Kailh_MX_Socket-compat"
+		(property "Footprint" "Library:hotswap"
 			(at 209.55 147.32 0)
 			(effects
@@
 			)
 		)
-		(property "Footprint" "keebio:Kailh_MX_Socket-compat"
+		(property "Footprint" "Library:hotswap"
 			(at 209.55 76.2 0)
 			(effects
@@
 			)
 		)
-		(property "Footprint" "keebio:Kailh_MX_Socket-compat"
+		(property "Footprint" "Library:hotswap"
 			(at 195.58 93.98 0)
 			(effects
